Commit message: [mod] modify joint/link name for easier understanding

File: code/models/humanModelTemplate/humanModelTemplate.urdf (robot description, URDF)
Before this commit: robot HumanModel, 103 links, 102 joints
Links:
- removed link C7Left_f1
- removed link C7Left_f2
- removed link C7Right_f1
- removed link C7Right_f2
- removed link L3
- removed link L3_f1
- removed link L5
- removed link L5_f1
- removed link T12
- removed link T12_f1
- removed link T8
- removed link T8_f1
- removed link T8_f2
- added link BottomLumbar, mass 1e-5; collision box size=1 1 1; visual box size=1 1 1
- added link BottomLumbar_f1, mass 1e-5
- added link Chest, mass 1e-5; collision box size=1 1 1; visual box size=1 1 1
- added link ChestLeft_f1, mass 1e-5
- added link ChestLeft_f2, mass 1e-5
- added link ChestRight_f1, mass 1e-5
- added link ChestRight_f2, mass 1e-5
- added link Chest_f1, mass 1e-5
- added link Chest_f2, mass 1e-5
- added link MidLumbar, mass 1e-5; collision box size=1 1 1; visual box size=1 1 1
- added link MidLumbar_f1, mass 1e-5
- added link TopLumbar, mass 1e-5; collision box size=1 1 1; visual box size=1 1 1
- added link TopLumbar_f1, mass 1e-5
Joints:
- removed joint jC1Head_rotx
- removed joint jC1Head_roty
- removed joint jC7LeftShoulder_rotx
- removed joint jC7LeftShoulder_roty
- removed joint jC7LeftShoulder_rotz
- removed joint jC7RightShoulder_rotx
- removed joint jC7RightShoulder_roty
- removed joint jC7RightShoulder_rotz
- removed joint jL1T12_rotx
- removed joint jL1T12_roty
- removed joint jL4L3_rotx
- removed joint jL4L3_roty
- removed joint jL5S1_rotx
- removed joint jL5S1_roty
- removed joint jT1C7_rotx
- removed joint jT1C7_roty
- removed joint jT1C7_rotz
- removed joint jT9T8_rotx
- removed joint jT9T8_roty
- removed joint jT9T8_rotz
- added joint jBottomLumbarMidLumbar_rotx: type revolute, parent BottomLumbar, child MidLumbar_f1, origin xyz=0 0 0 rpy=0 0 0, axis 1 0 0, limit lower=-0.610865 upper=0.610865 effort=30 velocity=1.0
- added joint jBottomLumbarMidLumbar_roty: type revolute, parent MidLumbar_f1, child MidLumbar, origin xyz=0 0 0 rpy=0 0 0, axis 0 1 0, limit lower=-0.523599 upper=1.309 effort=30 velocity=1.0
- added joint jBottomLumbarPelvis_rotx: type revolute, parent Pelvis, child BottomLumbar_f1, origin xyz=0 0 0 rpy=0 0 0, axis 1 0 0, limit lower=-0.610865 upper=0.610865 effort=30 velocity=1.0
- added joint jBottomLumbarPelvis_roty: type revolute, parent BottomLumbar_f1, child BottomLumbar, origin xyz=0 0 0 rpy=0 0 0, axis 0 1 0, limit lower=-0.523599 upper=1.309 effort=30 velocity=1.0
- added joint jChestLeftShoulder_rotx: type revolute, parent Chest, child ChestLeft_f1, origin xyz=0 0 0 rpy=0 0 0, axis 1 0 0, limit lower=-0.0872665 upper=0.785398 effort=30 velocity=1.0
- added joint jChestLeftShoulder_roty: type revolute, parent ChestLeft_f1, child ChestLeft_f2, origin xyz=0 0 0 rpy=0 0 0, axis 0 1 0, limit lower=-0.349066 upper=0.349066 effort=30 velocity=1.0
- added joint jChestLeftShoulder_rotz: type revolute, parent ChestLeft_f2, child LeftShoulder, origin xyz=0 0 0 rpy=0 0 0, axis 0 0 1, limit lower=-0.349066 upper=0.349066 effort=30 velocity=1.0
- added joint jChestRightShoulder_rotx: type revolute, parent Chest, child ChestRight_f1, origin xyz=0 0 0 rpy=0 0 0, axis 1 0 0, limit lower=-0.785398 upper=0.0872665 effort=30 velocity=1.0
- added joint jChestRightShoulder_roty: type revolute, parent ChestRight_f1, child ChestRight_f2, origin xyz=0 0 0 rpy=0 0 0, axis 0 1 0, limit lower=-0.349066 upper=0.349066 effort=30 velocity=1.0
- added joint jChestRightShoulder_rotz: type revolute, parent ChestRight_f2, child RightShoulder, origin xyz=0 0 0 rpy=0 0 0, axis 0 0 1, limit lower=-0.349066 upper=0.349066 effort=30 velocity=1.0
- added joint jMidLumbarTopLumbar_rotx: type revolute, parent MidLumbar, child TopLumbar_f1, origin xyz=0 0 0 rpy=0 0 0, axis 1 0 0, limit lower=-0.610865 upper=0.610865 effort=30 velocity=1.0
- added joint jMidLumbarTopLumbar_roty: type revolute, parent TopLumbar_f1, child TopLumbar, origin xyz=0 0 0 rpy=0 0 0, axis 0 1 0, limit lower=-0.523599 upper=1.309 effort=30 velocity=1.0
- added joint jNeckChest_rotx: type revolute, parent Chest, child Neck_f1, origin xyz=0 0 0 rpy=0 0 0, axis 1 0 0, limit lower=-0.610865 upper=0.610865 effort=30 velocity=1.0
- added joint jNeckChest_roty: type revolute, parent Neck_f1, child Neck_f2, origin xyz=0 0 0 rpy=0 0 0, axis 0 1 0, limit lower=-0.959931 upper=1.5708 effort=30 velocity=1.0
- added joint jNeckChest_rotz: type revolute, parent Neck_f2, child Neck, origin xyz=0 0 0 rpy=0 0 0, axis 0 0 1, limit lower=-1.22173 upper=1.22173 effort=30 velocity=1.0
- added joint jNeckHead_rotx: type revolute, parent Neck, child Head_f1, origin xyz=0 0 0 rpy=0 0 0, axis 1 0 0, limit lower=-0.610865 upper=0.610865 effort=30 velocity=1.0
- added joint jNeckHead_roty: type revolute, parent Head_f1, child Head, origin xyz=0 0 0 rpy=0 0 0, axis 0 1 0, limit lower=-0.436332 upper=0.174533 effort=30 velocity=1.0
- added joint jTopLumbarChest_rotx: type revolute, parent TopLumbar, child Chest_f1, origin xyz=0 0 0 rpy=0 0 0, axis 1 0 0, limit lower=-0.349066 upper=0.349066 effort=30 velocity=1.0
- added joint jTopLumbarChest_roty: type revolute, parent Chest_f1, child Chest_f2, origin xyz=0 0 0 rpy=0 0 0, axis 0 1 0, limit lower=-0.261799 upper=0.698132 effort=30 velocity=1.0
- added joint jTopLumbarChest_rotz: type revolute, parent Chest_f2, child Chest, origin xyz=0 0 0 rpy=0 0 0, axis 0 0 1, limit lower=-0.610865 upper=0.610865 effort=30 velocity=1.0
- joint jLeftErSpin_LUT: parent T8 -> Chest
- joint jLeftRecAbd_LUT: parent T8 -> Chest
- joint jRightErSpin_RUT: parent T8 -> Chest
- joint jRightRecAbd_RUT: parent T8 -> Chest
