Commit message: [mod] link name & link scale

File: code/models/female.urdf (robot description, URDF)
Before this commit: robot HumanModel, 103 links, 102 joints
Links:
- removed link Pelvis
- added link base, mass 6.9797; collision box size=0.225 0.318015 0.12987; visual mesh filename=meshes/base.stl scale=1. 1. 1.
Joints:
- removed joint jBottomLumbarPelvis_rotx
- removed joint jBottomLumbarPelvis_roty
- added joint jBottomLumbarbase_rotx: type revolute, parent base, child BottomLumbar_f1, origin xyz=0.0 0.0 0.064935 rpy=0.0 0.0 0.0, axis 1. 0. 0., limit lower=-0.610865 upper=0.610865 effort=30.0 velocity=1.0
- added joint jBottomLumbarbase_roty: type revolute, parent BottomLumbar_f1, child BottomLumbar, origin xyz=0.0 0.0 0.0 rpy=0.0 0.0 0.0, axis 0. 1. 0., limit lower=-0.523599 upper=1.309 effort=30.0 velocity=1.0
- joint jLeftErSpin_LP: parent Pelvis -> base
- joint jLeftHip_rotx: parent Pelvis -> base
- joint jLeftRecAbd_LP: parent Pelvis -> base
- joint jLeftRecFem_LP: parent Pelvis -> base
- joint jRightErSpin_RP: parent Pelvis -> base
- joint jRightHip_rotx: parent Pelvis -> base
- joint jRightRecAbd_RP: parent Pelvis -> base
- joint jRightRecFem_RP: parent Pelvis -> base

File: code/models/humanModelTemplate/humanModelTemplate.urdf (robot description, URDF)
Before this commit: robot HumanModel, 103 links, 102 joints
Links:
- removed link Pelvis
- added link base, mass 1e-5; collision box size=1 1 1; visual box size=1 1 1
Joints:
- removed joint jBottomLumbarPelvis_rotx
- removed joint jBottomLumbarPelvis_roty
- added joint jBottomLumbarbase_rotx: type revolute, parent base, child BottomLumbar_f1, origin xyz=0 0 0 rpy=0 0 0, axis 1 0 0, limit lower=-0.610865 upper=0.610865 effort=30 velocity=1.0
- added joint jBottomLumbarbase_roty: type revolute, parent BottomLumbar_f1, child BottomLumbar, origin xyz=0 0 0 rpy=0 0 0, axis 0 1 0, limit lower=-0.523599 upper=1.309 effort=30 velocity=1.0
- joint jLeftErSpin_LP: parent Pelvis -> base
- joint jLeftHip_rotx: parent Pelvis -> base
- joint jLeftRecAbd_LP: parent Pelvis -> base
- joint jLeftRecFem_LP: parent Pelvis -> base
- joint jRightErSpin_RP: parent Pelvis -> base
- joint jRightHip_rotx: parent Pelvis -> base
- joint jRightRecAbd_RP: parent Pelvis -> base
- joint jRightRecFem_RP: parent Pelvis -> base
